File: phase-driver.kicad_sch (KiCad schematic)
At the start: 13 parts, among them Q1 LMG2100R026, U1 MCS1823

Commit message: fix: adjusted positining
Changed lines of the file:
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@@
 	(wire
 		(pts
-			(xy 171.45 78.74) (xy 237.49 78.74)
-		)
-		(stroke
-			(width 0)
-			(type default)
-		)
-	)
-	(wire
-		(pts
-			(xy 163.83 148.59) (xy 171.45 148.59)
+			(xy 181.61 78.74) (xy 237.49 78.74)
+		)
+		(stroke
+			(width 0)
+			(type default)
+		)
+	)
+	(wire
+		(pts
+			(xy 163.83 148.59) (xy 181.61 148.59)
 		)
 		(stroke
@@
 	(wire
 		(pts
-			(xy 171.45 148.59) (xy 171.45 78.74)
+			(xy 181.61 148.59) (xy 181.61 78.74)
 		)
 		(stroke
@@
 	)
 	(label "PH_OUT"
-		(at 173.99 78.74 0)
+		(at 181.61 78.74 0)
 		(effects
 			(font
